Commit message: Add Lidar Sensor to the robot

File: urdf/jetracer.xacro (robot description, xacro)
@@ -161,4 +161,31 @@
     <origin xyz="0 0 0" rpy="0 0 0"/>
   </joint>
+  <!-- Lidar -->
+  <link name="laser_link">
+    <inertial>
+      <mass value="0.1"/>
+      <origin xyz="0 0 0" rpy="0 0 0"/>
+      <inertia ixx="0.001" ixy="0" ixz="0"
+               iyy="0.001" iyz="0" izz="0.001"/>
+    </inertial>
+    <visual>
+      <origin xyz="0 0 0" rpy="0 0 0"/>
+      <geometry>
+        <cylinder radius="0.04" length="0.06"/>
+      </geometry>
+      <material name="red"/>
+    </visual>
+    <collision>
+      <origin xyz="0 0 0" rpy="0 0 0"/>
+      <geometry>
+        <cylinder radius="0.04" length="0.06"/>
+      </geometry>
+    </collision>
+  </link>
+  <joint name="laser_joint" type="fixed">
+    <parent link="chassis"/>
+    <child link="laser_link"/>
+    <origin xyz="0 0 ${chassis_height/2 + 0.08}" rpy="0 0 0"/>
+  </joint>
   <!-- Gazebo specific configurations -->
   <gazebo reference="chassis">
@@ -209,4 +236,35 @@
     </sensor>
   </gazebo>
+  <gazebo reference="laser_link">
+    <material>Gazebo/Red</material>
+    <sensor type="gpu_lidar" name="laser">
+      <update_rate>10</update_rate>
+      <topic>/scan</topic>
+      <ray>
+        <scan>
+          <horizontal>
+            <samples>360</samples>
+            <resolution>1</resolution>
+            <min_angle>-3.14159</min_angle>
+            <max_angle>3.14159</max_angle>
+          </horizontal>
+          <vertical>
+            <samples>1</samples>
+            <resolution>1</resolution>
+            <min_angle>0</min_angle>
+            <max_angle>0</max_angle>
+          </vertical>
+        </scan>
+        <range>
+          <min>0.1</min>
+          <max>10.0</max>
+          <resolution>0.01</resolution>
+        </range>
+      </ray>
+      <plugin filename="gz-sim-sensors-system" name="gz::sim::systems::Sensors">
+        <render_engine>ogre2</render_engine>
+      </plugin>
+    </sensor>
+  </gazebo>
   <!-- Ackermann steering plugin for Gazebo Harmonic -->
   <gazebo>
